File: AD4DA-LightUI.brd (EAGLE design)
At the start: 106 x 100 mm, 13 parts

Commit message: 2.0
Parts:
- removed C4, C5: 0.1uF, SPCoast:C050-024X044
- removed LED1: WHITE, SPCoast:LED5MM
- removed R1: 1k0, SPCoast:AXIAL-0.3-RES
- added JP1: (no value), SPCoast:1X03
- C1, C2: value 150uF -> 0.1uF; device SPCoast:E5-10.5 -> SPCoast:C050-024X044
- U$1: value SLIDE-POT-45MM -> R-SLIDE-POT-45MM; device SPCoast:SLIDER-45MM-LARGE -> SPCoast:SLIDER-45MM
- U$2, U$3, U$7: value (none) -> R-SLIDE-POT-45MM; device SPCoast:SLIDER-45MM-LARGE -> SPCoast:SLIDER-45MM
- moved C2 72.0 mm to (15.9, 55.2)
- moved U$1 6.35 mm to (40.0, 46.4)
- moved U$2 6.35 mm to (48.9, 46.4)
- moved U$3 6.35 mm to (57.8, 46.4)
- moved U$7 5.99 mm to (75.6, 46.4)
- moved C1 5.75 mm to (21.0, 55.2)
- moved X1 3.59 mm to (20.3, 86.4)
Connections:
- removed net N$2: LED1.K, R1.P$1
- net 5V: now also C1.1, C2.1, JP1.1; no longer C1.+, C2.+, C4.1, C5.1
- net AGND: now also C1.2, JP1.3; no longer C1.-, C2.-, C4.2, C5.2
- net DA0: now also JP1.2; no longer LED1.A
- net GND: now also C2.2; no longer R1.P$2
Routing:
- net AGND: track 0.00 -> 84.8 mm
- net GND: track 91.4 -> 30.5 mm
- net AD0: track 56.1 -> 79.4 mm
- net DA0: track 70.1 -> 55.2 mm
- net AD2: track 31.3 -> 40.5 mm
- net AD1: track 41.1 -> 48.4 mm
- net N$2: track 6.35 -> 0.00 mm
- net AD3: track 26.4 -> 29.4 mm
Other:
- board text added: "2014-11 B"
- board text added: "OSHW John Plocher"
- board text added: "Slide pot had incorrect pin spacing"
- board text added: "v2.0"
- board text removed: "2014-10 A"
- board text removed: "OSHW"
- board text removed: "v1.0"

Commit message: 2.1
Parts:
- JP1: value (none) -> JUMPER-3PTH-LOCK
- renumbered U$9 to BOARD1
Routing:
- net AD0: track 79.4 -> 71.8 mm
Other:
- board text added: "2014-12 C"
- board text added: "OSHW"
- board text added: "Silk Screen mixed AGND and +5V labels"
- board text added: "v2.1"
- board text removed: "2014-11 B"
- board text removed: "OSHW John Plocher"
- board text removed: "Slide pot had incorrect pin spacing"
- board text removed: "v2.0"
Changed lines of the file:
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@@
 <text x="39.18" y="82.68" size="2.54" layer="51">R   G   B </text>
 <text x="72.09" y="82.68" size="2.54" layer="51">White</text>
-<text x="94.945" y="53.54" size="2.54" layer="51" ratio="15" rot="R90">LightUI</text>
+<text x="97.485" y="67.51" size="2.54" layer="51" ratio="15" rot="R90">LightUI</text>
 <text x="60.96" y="86.36" size="1.4224" layer="51">D/A out</text>
-<text x="93.18333125" y="88.646" size="1.27" layer="51" rot="SR0">v2.0</text>
-<text x="1.10833125" y="79.121" size="1.016" layer="51" ratio="10" rot="SR0">   OSHW
-John Plocher</text>
+<text x="93.18333125" y="88.646" size="1.27" layer="51" rot="SR0">v2.1</text>
+<text x="1.10833125" y="79.121" size="1.016" layer="51" ratio="10" rot="SR0">   OSHW</text>
 <text x="25.4" y="71.12" size="1.016" layer="51" rot="R90">+5</text>
 <text x="19.05" y="70.485" size="1.016" layer="51" rot="R90">Agnd</text>
@@
 <text x="78.74" y="77.47" size="1.016" layer="51" rot="R90">AD0</text>
 <text x="59.69" y="77.47" size="1.016" layer="51" rot="R90">AD1</text>
-<text x="50.8" y="81.28" size="1.016" layer="51" rot="R90">AD2</text>
+<text x="50.8" y="77.47" size="1.016" layer="51" rot="R90">AD2</text>
 <text x="43.18" y="77.47" size="1.016" layer="51" rot="R90">AD3</text>
 <text x="67.31" y="77.47" size="1.016" layer="51" rot="R90">DA0</text>
@@
 <text x="69.85" y="76.835" size="1.016" layer="51" rot="R90">Agnd</text>
 <text x="64.77" y="78.105" size="1.016" layer="51" rot="R90">+5</text>
-<text x="-2.54" y="27.94" size="1.778" layer="102" rot="R90">Slide pot had incorrect pin spacing</text>
-<text x="88.10333125" y="20.066" size="1.016" layer="51" rot="SR0">2014-11 B</text>
-<text x="10.795" y="45.72" size="2.54" layer="51" rot="R180">Agnd</text>
-<text x="6.35" y="70.485" size="2.54" layer="51" rot="R180">+5</text>
+<text x="-2.54" y="27.94" size="1.778" layer="102" rot="R90">Silk Screen mixed AGND and +5V labels</text>
+<text x="10.795" y="71.12" size="2.54" layer="51" rot="R180">Agnd</text>
+<text x="7.62" y="45.085" size="2.54" layer="51" rot="R180">+5</text>
+<text x="88.10333125" y="20.066" size="1.016" layer="51" rot="SR0">2014-12 C</text>
 </plain>
 <attributes>
@@
 <element name="U$3" library="SPCoast" package="SLIDER-45MM" value="R-SLIDE-POT-45MM" x="57.785" y="46.355" rot="R270"/>
 <element name="U$7" library="SPCoast" package="SLIDER-45MM" value="R-SLIDE-POT-45MM" x="75.565" y="46.355" rot="R270"/>
-<element name="U$9" library="SPCoast" package="BOARD-DINRAIL-3.17INX10CM" value="BOARD80X100" x="0" y="0"/>
 <element name="C1" library="SPCoast" package="C050-024X044" value="0.1uF" x="20.955" y="55.245" smashed="yes" rot="R90">
 <attribute name="NAME" x="19.4945" y="54.483" size="1.016" layer="25" rot="R90"/>
@@
 <element name="LOGO1" library="SPCoast" package="OSHW-LOGO-L" value="DOC-OSHW-LOGO-L" x="5.08" y="85.09"/>
 <element name="C2" library="SPCoast" package="C050-024X044" value="0.1uF" x="15.875" y="55.245" rot="R90"/>
-<element name="JP1" library="SPCoast" package="1X03" value="" x="64.135" y="82.55" smashed="yes">
+<element name="JP1" library="SPCoast" package="1X03" value="JUMPER-3PTH-LOCK" x="64.135" y="82.55" smashed="yes">
 <attribute name="NAME" x="62.7888" y="84.3788" size="1.27" layer="25" ratio="10"/>
 </element>
+<element name="BOARD1" library="SPCoast" package="BOARD-DINRAIL-3.17INX10CM" value="BOARD80X100" x="0" y="0"/>
 </elements>
 <signals>
@@
 <contactref element="C1" pad="1"/>
 <polygon width="0.4064" layer="1" isolate="0.6096">
-<vertex x="0" y="89.408"/>
-<vertex x="100.076" y="89.408"/>
-<vertex x="100.076" y="11.43"/>
-<vertex x="0" y="11.43"/>
+<vertex x="0" y="90.16"/>
+<vertex x="100" y="90.16"/>
+<vertex x="100" y="10.16"/>
+<vertex x="0" y="10.16"/>
 </polygon>
 <contactref element="X1" pad="1"/>
@@
 <wire x1="75.3" y1="68.58" x2="53.975" y2="68.58" width="0.4064" layer="16"/>
 <wire x1="53.975" y1="68.58" x2="53.34" y2="69.215" width="0.4064" layer="16"/>
-<wire x1="53.34" y1="69.215" x2="53.34" y2="76.2" width="0.4064" layer="16"/>
-<wire x1="53.34" y1="76.2" x2="52.07" y2="77.47" width="0.4064" layer="16"/>
-<wire x1="52.07" y1="77.47" x2="45.085" y2="77.47" width="0.4064" layer="16"/>
-<wire x1="45.085" y1="77.47" x2="44.45" y2="76.835" width="0.4064" layer="16"/>
-<wire x1="44.45" y1="76.835" x2="44.45" y2="69.215" width="0.4064" layer="16"/>
+<wire x1="53.34" y1="69.215" x2="53.34" y2="72.39" width="0.4064" layer="16"/>
+<wire x1="53.34" y1="72.39" x2="52.07" y2="73.66" width="0.4064" layer="16"/>
+<wire x1="52.07" y1="73.66" x2="45.085" y2="73.66" width="0.4064" layer="16"/>
+<wire x1="45.085" y1="73.66" x2="44.45" y2="73.025" width="0.4064" layer="16"/>
+<wire x1="44.45" y1="73.025" x2="44.45" y2="69.215" width="0.4064" layer="16"/>
 <wire x1="44.45" y1="69.215" x2="43.815" y2="68.58" width="0.4064" layer="16"/>
 <wire x1="43.815" y1="68.58" x2="24.765" y2="68.58" width="0.4064" layer="16"/>
@@
 <contactref element="C1" pad="2"/>
 <polygon width="0.4064" layer="16" isolate="0.4064">
-<vertex x="0" y="89.408"/>
-<vertex x="100.076" y="89.408"/>
-<vertex x="100.076" y="11.43"/>
-<vertex x="0" y="11.43"/>
+<vertex x="0" y="90.16"/>
+<vertex x="100" y="90.16"/>
+<vertex x="100" y="10.16"/>
+<vertex x="0" y="10.16"/>
 </polygon>
 <via x="5.08" y="73.66" extent="1-16" drill="3.2" shape="octagon"/>
@@
 </board>
 </drawing>
-<compatibility>
-<note version="6.3" minversion="6.2.2" severity="warning">
-Since Version 6.2.2 text objects can contain more than one line,
-which will not be processed correctly with this version.
-</note>
-</compatibility>
 </eagle>

Commit message: 2.2
Parts:
- removed U$1, U$2, U$3, U$7: R-SLIDE-POT-45MM, SPCoast:SLIDER-45MM
- added RS1, RS2, RS3, RS4: 10K OHM "B" TAPER, SPCoast:SLIDER-45MM
- BOARD1: value BOARD80X100 -> 10x7cm; device SPCoast:BOARD-DINRAIL-3.17INX10CM -> SPCoast:BOARD-DINRAIL-3.17INX7CM
- JP1: value JUMPER-3PTH-LOCK -> 1x3
- X1: value (none) -> RJ45/8
- moved LOGO1 69.9 mm to (5.08, 15.2)
- moved JP1 61.7 mm to (7.62, 57.8), turned to 90 degrees
- moved C2 22.2 mm to (6.99, 75.6), turned to 270 degrees
- moved C1 11.4 mm to (10.8, 60.3)
- moved X1 4.02 mm to (16.5, 85.1)
Connections:
- net 5V: now also RS1.E, RS2.E, RS3.E, RS4.E; no longer U$1.E, U$2.E, U$3.E, U$7.E
- net AD0: now also RS4.S; no longer U$7.S
- net AD1: now also RS3.S; no longer U$3.S
- net AD2: now also RS2.S; no longer U$2.S
- net AD3: now also RS1.S; no longer U$1.S
- net AGND: now also RS1.A, RS1.AGND@0, RS1.AGND@1, RS2.A, RS2.AGND@0, RS2.AGND@1, RS3.A, RS3.AGND@0, RS3.AGND@1, RS4.A, RS4.AGND@0, RS4.AGND@1; no longer U$1.A, U$2.A, U$3.A, U$7.A
Routing:
- net AGND: track 84.8 -> 0.00 mm, vias 1 -> 0
- net GND: track 30.5 -> 7.51 mm, vias 1 -> 0
- net DA0: track 55.2 -> 32.7 mm
- net AD2: track 40.5 -> 32.9 mm
- net AD3: track 29.4 -> 21.8 mm
- net AD1: track 48.4 -> 41.6 mm
- net AD0: track 71.8 -> 65.4 mm
Other:
- board size 106 x 100 mm -> 76 x 100 mm
- board text added: "2018-07"
- board text added: "Shrunk board size"
- board text added: "W"
- board text added: "v1.0D"
- board text added: "v2.2"
- board text removed: "2014-12 C"
- board text removed: "Silk Screen mixed AGND and +5V labels"
- board text removed: "White"
- board text removed: "v2.1"
