File: AD4DA-LightUI.sch (EAGLE design)
At the start: 13 parts

Commit message: 2.0
Parts:
- removed C4, C5: 0.1uF, SPCoast:CAPPTH1
- removed LED1: WHITE, SPCoast:LEDLED5MM
- removed R1: 1k0, SPCoast:RPTH03
- added JP1: (no value), SPCoast:JUMPER-3PTH-LOCK
- C1, C2: value 150uF -> 0.1uF; device SPCoast:CAP-POLPTH-5MM -> SPCoast:CAPPTH1
- U$1: value SLIDE-POT-45MM -> R-SLIDE-POT-45MM; device SPCoast:R-SLIDE-POT -> SPCoast:R-SLIDE-POT-45MM
- U$2, U$3, U$7: value (none) -> R-SLIDE-POT-45MM; device SPCoast:R-SLIDE-POT -> SPCoast:R-SLIDE-POT-45MM
Connections:
- removed net N$2: LED1.C, R1.1
- net 5V: now also C1.1, C2.1, JP1.1, U$1.E, U$2.E, U$3.E, U$7.E; no longer C1.+, C2.+, C4.1, C5.1, U$1RS1.E, U$2RS1.E, U$3RS1.E, U$7RS1.E
- net AD0: now also U$7.S; no longer U$7RS1.S
- net AD1: now also U$3.S; no longer U$3RS1.S
- net AD2: now also U$2.S; no longer U$2RS1.S
- net AD3: now also U$1.S; no longer U$1RS1.S
- net AGND: now also C1.2, JP1.3, U$1.A, U$2.A, U$3.A, U$7.A; no longer C1.-, C2.-, C4.2, C5.2, U$1RS1.A, U$2RS1.A, U$3RS1.A, U$7RS1.A
- net DA0: now also JP1.2; no longer LED1.A
- net GND: now also C2.2; no longer R1.2
Other:
- note added: "2.0"
- note added: "Update: Fixed library footprint for sliders removed extra caps analog output to a pin set, not LED"
- note removed: "1.0"

Commit message: 2.1
Parts:
- removed U$9: BOARD80X100, SPCoast:BOARD80X100
- added BOARD1: BOARD80X100, SPCoast:BOARD80X100
- C1, C2: device SPCoast:CAPPTH1 -> SPCoast:CAP
- JP1: value (none) -> JUMPER-3PTH-LOCK
Other:
- note added: "2.1"
- note added: "C"
- note removed: "2.0"
- note removed: "A"
Changed lines of the file:
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@@
 <part name="U$3" library="SPCoast" deviceset="R-SLIDE-POT" device="-45MM"/>
 <part name="U$7" library="SPCoast" deviceset="R-SLIDE-POT" device="-45MM"/>
-<part name="U$9" library="SPCoast" deviceset="BOARD" device="80X100" value="BOARD80X100"/>
 <part name="SUPPLY4" library="SparkFun-Aesthetics" deviceset="5V" device=""/>
 <part name="SUPPLY8" library="SparkFun-Aesthetics" deviceset="5V" device=""/>
 <part name="SUPPLY9" library="SparkFun-Aesthetics" deviceset="5V" device=""/>
 <part name="SUPPLY10" library="SparkFun-Aesthetics" deviceset="5V" device=""/>
-<part name="C1" library="SPCoast" deviceset="CAP*" device="PTH1" value="0.1uF"/>
+<part name="C1" library="SPCoast" deviceset="CAP*" device="" value="0.1uF"/>
 <part name="SUPPLY13" library="SparkFun-Aesthetics" deviceset="5V" device=""/>
 <part name="X1" library="SPCoast" deviceset="CONNECTOR-RJ45" device="-FRONT"/>
@@
 <part name="GND10" library="SparkFun-Aesthetics" deviceset="GND" device=""/>
 <part name="LOGO1" library="SPCoast" deviceset="DOC-OSHW-LOGO-" device="L"/>
-<part name="C2" library="SPCoast" deviceset="CAP*" device="PTH1" value="0.1uF"/>
+<part name="C2" library="SPCoast" deviceset="CAP*" device="" value="0.1uF"/>
 <part name="GND1" library="SparkFun-Aesthetics" deviceset="GND" device=""/>
 <part name="JP1" library="SPCoast" deviceset="JUMPER-3" device="PTH-LOCK"/>
 <part name="SUPPLY1" library="SparkFun-Aesthetics" deviceset="5V" device=""/>
+<part name="BOARD1" library="SPCoast" deviceset="BOARD" device="80X100"/>
 </parts>
 <sheets>
@@
 <plain>
 <text x="149.86" y="20.32" size="2.54" layer="97">4x slider pots for controlling light strips</text>
-<text x="238.76" y="12.7" size="2.54" layer="95">2.0</text>
-<text x="239.268" y="6.35" size="2.54" layer="95">A</text>
+<text x="238.76" y="12.7" size="2.54" layer="95">2.1</text>
+<text x="239.268" y="6.35" size="2.54" layer="95">C</text>
 <text x="5.08" y="2.54" size="2.54" layer="95">Update:  Fixed library footprint for sliders
 removed extra caps
@@
 <instance part="U$3" gate="P1" x="68.58" y="134.62"/>
 <instance part="U$7" gate="P1" x="99.06" y="134.62"/>
-<instance part="U$9" gate="B" x="132.08" y="10.16"/>
 <instance part="SUPPLY4" gate="G$1" x="99.06" y="142.24"/>
 <instance part="SUPPLY8" gate="G$1" x="68.58" y="142.24"/>
 <instance part="SUPPLY9" gate="G$1" x="50.8" y="142.24"/>
 <instance part="SUPPLY10" gate="G$1" x="33.02" y="142.24"/>
-<instance part="C1" gate="C1" x="119.38" y="132.08"/>
+<instance part="C1" gate="G$1" x="119.38" y="132.08"/>
 <instance part="SUPPLY13" gate="G$1" x="129.54" y="137.16"/>
 <instance part="X1" gate="J" x="213.36" y="111.76"/>
@@
 <instance part="GND10" gate="1" x="210.82" y="96.52"/>
 <instance part="LOGO1" gate="DOC-OSHW-LOGO" x="132.08" y="25.4"/>
-<instance part="C2" gate="C1" x="139.7" y="132.08"/>
+<instance part="C2" gate="G$1" x="139.7" y="132.08"/>
 <instance part="GND1" gate="1" x="139.7" y="124.46"/>
-<instance part="JP1" gate="J" x="53.34" y="104.14" rot="R270"/>
+<instance part="JP1" gate="G$1" x="53.34" y="104.14" rot="R270"/>
 <instance part="SUPPLY1" gate="G$1" x="50.8" y="104.14"/>
+<instance part="BOARD1" gate="B" x="132.08" y="7.62"/>
 </instances>
 <busses>
@@
 </segment>
 <segment>
-<pinref part="C1" gate="C1" pin="1"/>
+<pinref part="C1" gate="G$1" pin="1"/>
 <wire x1="119.38" y1="134.62" x2="129.54" y2="134.62" width="0.1524" layer="91"/>
 <junction x="129.54" y="134.62"/>
@@
 <pinref part="SUPPLY13" gate="G$1" pin="5V"/>
 <wire x1="129.54" y1="134.62" x2="139.7" y2="134.62" width="0.1524" layer="91"/>
-<pinref part="C2" gate="C1" pin="1"/>
+<pinref part="C2" gate="G$1" pin="1"/>
 </segment>
 <segment>
@@
 </segment>
 <segment>
-<pinref part="JP1" gate="J" pin="1"/>
+<pinref part="JP1" gate="G$1" pin="1"/>
 <pinref part="SUPPLY1" gate="G$1" pin="5V"/>
 </segment>
@@
 </segment>
 <segment>
-<pinref part="C2" gate="C1" pin="2"/>
+<pinref part="C2" gate="G$1" pin="2"/>
 <pinref part="GND1" gate="1" pin="GND"/>
 </segment>
@@
 <segment>
 <wire x1="50.8" y1="101.6" x2="45.72" y2="101.6" width="0.1524" layer="91"/>
-<pinref part="JP1" gate="J" pin="2"/>
+<pinref part="JP1" gate="G$1" pin="2"/>
 <label x="45.72" y="101.6" size="1.4224" layer="95" rot="R180" xref="yes"/>
 </segment>
@@
 <junction x="99.06" y="127"/>
 <label x="99.06" y="121.92" size="1.016" layer="95" rot="R270" xref="yes"/>
-<pinref part="C1" gate="C1" pin="2"/>
+<pinref part="C1" gate="G$1" pin="2"/>
 <junction x="119.38" y="127"/>
 <wire x1="99.06" y1="127" x2="119.38" y2="127" width="0.1524" layer="91"/>
@@
 </segment>
 <segment>
-<pinref part="JP1" gate="J" pin="3"/>
+<pinref part="JP1" gate="G$1" pin="3"/>
 <wire x1="50.8" y1="99.06" x2="50.8" y2="93.98" width="0.1524" layer="91"/>
 <label x="50.8" y="93.98" size="1.4224" layer="95" xref="yes"/>

Commit message: 2.2
Parts:
- removed U$1, U$2, U$3, U$7: R-SLIDE-POT-45MM, SPCoast:R-SLIDE-POT-45MM
- added RS1, RS2, RS3, RS4: 10K OHM "B" TAPER, SPCoast:R-SLIDE-POT-45MM
- BOARD1: value BOARD80X100 -> 10x7cm; device SPCoast:BOARD80X100 -> SPCoast:BOARD80X70
- C1, C2: device SPCoast:CAP -> SPCoast:CAPPTH1
- JP1: value JUMPER-3PTH-LOCK -> 1x3
- X1: value (none) -> RJ45/8
Connections:
- net 5V: now also RS1RS1.E, RS2RS1.E, RS3RS1.E, RS4RS1.E; no longer U$1.E, U$2.E, U$3.E, U$7.E
- net AD0: now also RS4RS1.S; no longer U$7.S
- net AD1: now also RS3RS1.S; no longer U$3.S
- net AD2: now also RS2RS1.S; no longer U$2.S
- net AD3: now also RS1RS1.S; no longer U$1.S
- net AGND: now also RS1G1.AGND, RS1RS1.A, RS2G1.AGND, RS2RS1.A, RS3G1.AGND, RS3RS1.A, RS4G1.AGND, RS4RS1.A; no longer U$1.A, U$2.A, U$3.A, U$7.A
Other:
- note added: "2.2"
- note added: "D"
- note removed: "2.1"
- note removed: "C"
- moved on the sheet: X1
